File: PlantSensor.kicad_pcb (KiCad board)
At the start: 2 copper layers, 70 x 70 mm, 51 parts, among them J1 SCREW-TERMINAL-GREEN_2P-5.0_, J2 SCREW-TERMINAL-GREEN_2P-5.0_, J3 SCREW-TERMINAL-GREEN_2P-5.0_, J4 SCREW-TERMINAL-GREEN_2P-5.0_, J5 DIP-BLACK-MALE-HEADER-VERT_2P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, J6 DIP-BLACK-MALE-HEADER-VERT_4P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, Q1 N-Channel_30-V_MOSFET, Q2 N-Channel_30-V_MOSFET, Q3 N-Channel_30-V_MOSFET, Q4 N-Channel_30-V_MOSFET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

Commit message: fixed trace size + diode to prevent inductive load from damaging the mosfet
Parts:
- added D1: DIODE, Diode_SMD:D_SOD-123, F.Cu at (166.0, 57.0)
- added D2: DIODE, Diode_SMD:D_SOD-123, F.Cu at (166.0, 72.0)
- added D3: DIODE, Diode_SMD:D_SOD-123, F.Cu at (166.0, 87.5)
- U11: value TEM-HUM-DHT11 -> TEM-HUM-DHT11_4P-15.5X12.0MM_
- moved J4 8.00 mm to (166.0, 80.0)
- moved J3 4.00 mm to (166.0, 65.0)
- moved BZ1 0.71 mm to (163.5, 92.7)
- moved J1 0.50 mm to (166.0, 38.5)
- moved J5 0.50 mm to (152.0, 38.5)
Routing:
- net +12V: track 97.0 -> 167.8 mm
- net GND: track 207.3 -> 264.0 mm, vias 6 -> 10
- net Net-(D3-Pad1): track 8.18 -> 21.2 mm
- net Net-(D2-Pad1): track 8.18 -> 16.3 mm
- net Net-(D1-Pad1): track 8.23 -> 11.9 mm
